File: PMB/PCB/PMB.brd (EAGLE design)
At the start: 125 x 57 mm, 96 parts, among them Q1 CRYSTAL_SM49, SW1 MC32829, U6 ATMEGA328P-AU, X1 16MHz

Commit message: Updated to latest PCB revision
Parts:
- removed D3, TXO: BLUE, SparkFun-LED:LED-0603
- removed R36: 100, resistor:R0805W
- added POWER: blue, Discrete:LED-0805
- added TX0: Blue, Discrete:LED-0805
- C2: value 150UF -> 100UF
- C3: value 22p -> 100p
- RXI, RX_CAN: value GREEN -> Green; device SparkFun-LED:LED-0603 -> Discrete:LED-0805
- TX_CAN: value BLUE -> Blue; device SparkFun-LED:LED-0603 -> Discrete:LED-0805
- WARNING: value RED -> (none); device SparkFun-LED:LED-0603 -> Discrete:LED-0805
- moved RX_CAN 2.03 mm to (115.8, 43.9), turned to 180 degrees
- moved N-MOS1 1.80 mm to (38.9, 45.7)
- moved RLY1 1.55 mm to (27.4, 48.5)
- moved C2 1.52 mm to (57.1, 48.3)
- moved D1 1.52 mm to (38.9, 51.6)
- moved R2 1.52 mm to (23.1, 48.5)
- moved RF1 1.30 mm to (38.9, 45.7)
- moved PMOS1 1.27 mm to (32.5, 38.1)
- moved R3 1.27 mm to (65.8, 27.9)
- moved R6 1.27 mm to (38.4, 40.4)
- moved RXI 1.05 mm to (102.1, 8.89), turned to 90 degrees
- moved TX_CAN 0.36 mm to (115.8, 40.1), turned to 180 degrees
- moved WARNING 0.28 mm to (71.9, 37.2), turned to 90 degrees
Connections:
- removed net SMF: R36.1, RLY1.12, RLY1.9
- net D0/RXI: now also RXI.-; no longer RXI.C
- net D1/TXO: now also TX0.-; no longer TXO.C
- net D2: now also WARNING.-; no longer WARNING.C
- net GND: now also POWER.-; no longer D3.C
- net N$10: now also WARNING.+; no longer WARNING.A
- net N$11: now also RXI.+; no longer RXI.A
- net N$12: now also TX0.+; no longer TXO.A
- net N$13: now also RX_CAN.+; no longer RX_CAN.A
- net N$14: now also TX_CAN.+; no longer TX_CAN.A
- net N$7: now also POWER.+; no longer D3.A
- net PE: now also RLY1.12, RLY1.9; no longer R36.2
- net RXCAN: now also RX_CAN.-; no longer RX_CAN.C
- net TXCAN: now also TX_CAN.-; no longer TX_CAN.C
Routing:
- net PE: track 130.1 -> 152.4 mm
- net SMF: track 18.5 -> 0.00 mm
- net GND: track 395.4 -> 406.9 mm, vias 62 -> 64
- net RLY7: track 11.1 -> 15.0 mm
- net N$12: track 2.67 -> 6.38 mm
- net VCC: track 86.3 -> 89.7 mm
- net RXCAN: track 36.1 -> 33.9 mm
- net N$13: track 6.46 -> 4.55 mm
- net PNP_GATE: track 21.0 -> 22.3 mm
- net GATE: track 53.3 -> 52.1 mm
- net N$11: track 3.09 -> 4.27 mm
- net D0/RXI: track 55.1 -> 54.0 mm
- net N$7: track 2.16 -> 3.18 mm
- net +24V: track 9.00 -> 9.95 mm
- net D1/TXO: track 55.8 -> 55.0 mm
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