File: PMB/PCB/PMB.sch (EAGLE design)
At the start: 96 parts, among them Q1 CRYSTAL_SM49, SW1 MC32829, U6 ATMEGA328P-AU, X1 16MHz

Commit message: Updated to latest PCB revision
Parts:
- removed D3, TXO: BLUE, SparkFun-LED:LED-BLUE0603
- removed R36: 100, resistor:R-EU_R0805W
- added POWER: blue, Discrete:LED-0805
- added TX0: Blue, Discrete:LED-0805
- C2: value 150UF -> 100UF
- C3: value 22p -> 100p
- RXI, RX_CAN: value GREEN -> Green; device SparkFun-LED:LED-GREEN0603 -> Discrete:LED-0805
- TX_CAN: value BLUE -> Blue; device SparkFun-LED:LED-BLUE0603 -> Discrete:LED-0805
- WARNING: value RED -> (none); device SparkFun-LED:LED-RED0603 -> Discrete:LED-0805
Connections:
- removed net SMF: R36.1, RLY1.12, RLY1.9
- net D0/RXI: now also RXI.-; no longer RXI.C
- net D1/TXO: now also TX0.-; no longer TXO.C
- net D2: now also WARNING.-; no longer WARNING.C
- net GND: now also POWER.-; no longer D3.C
- net N$10: now also WARNING.+; no longer WARNING.A
- net N$11: now also RXI.+; no longer RXI.A
- net N$12: now also TX0.+; no longer TXO.A
- net N$13: now also RX_CAN.+; no longer RX_CAN.A
- net N$14: now also TX_CAN.+; no longer TX_CAN.A
- net N$7: now also POWER.+; no longer D3.A
- net PE: now also RLY1.12, RLY1.9; no longer R36.2
- net RXCAN: now also RX_CAN.-; no longer RX_CAN.C
- net TXCAN: now also TX_CAN.-; no longer TX_CAN.C
