File: AUV/PMB/PCB/PMB.brd (EAGLE design)
At the start: 125 x 57 mm, 95 parts, among them Q1 CRYSTAL_SM49, SW1 MC32829, U6 ATMEGA328P-AU, X1 16MHz

Commit message: Shifted libraries to same folder as main code. Calibration files updated for PMB1,2,3,4,5,6.
Parts:
- C3: value 100p -> 100n
